File: HackPad.kicad_pcb (KiCad board)
At the start: 2 copper layers, 92.9 x 46.9 mm, 7 parts, among them SW1 SW_Push, SW2 SW_Push, SW3 SW_Push, SW4 SW_Push, SW5 SW_Push, SW6 SW_Push, U1 XIAO-RP2040-DIP

Commit message: Added PCB, main.py
Parts:
- added G***: LOGO, LOGO, F.Cu at (69.4, 95.4)
- added G***: LOGO, LOGO, F.Cu at (34.4, 80.6)
- moved U1 12.9 mm to (63.7, 77.1), turned to 90 degrees
Routing:
- net GND: track 116.5 -> 142.2 mm
- net Net-(U1-GPIO3/MOSI): track 65.7 -> 82.1 mm
- net Net-(U1-GPIO0/TX): track 33.8 -> 18.1 mm
- net Net-(U1-GPIO4/MISO): track 54.8 -> 66.9 mm
- net Net-(U1-GPIO2/SCK): track 38.3 -> 45.9 mm
- net Net-(U1-GPIO1/RX): track 35.2 -> 41.3 mm
- net Net-(U1-GPIO7/SCL): track 30.4 -> 31.6 mm
